File: Hardware/KiCAD/JumperlessRev3point1/JumperlessRev3point1.kicad_sch (KiCad schematic)
At the start: 207 parts, among them J1 Debug, J14 5V, J4 Breadboard, J5 USB_B_Mini, J6 CH446Q, J7 Conn_01x04_Pin, K1 CH446Q, SW1 USB BOOT, SW2 SW_DP3T, U1 LT1054, U10 L272D, U11 LM324, U12 MCP4822, U2 NCP1117-3.3_SOT223, U4 INA219, U6 INA219, U7 LM324, U8 W25Q128JVS, U9 RP2040, Y1 ABLS-12.000MHZ-B4-T

Commit message: Added contact info and stuff to be super duper open source
Other:
- company: (none) -> Architeuthis Flux
- title: (none) -> Jumperless Rev 3.1
Changed lines of the file:
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@@
 	(generator_version "8.0")
 	(paper "A1")
+	(title_block
+		(title "Jumperless Rev 3.1")
+		(date "2023-11-11")
+		(rev "3.1")
+		(company "Architeuthis Flux")
+		(comment 1 "Kevin Santo Cappuccio")
+		(comment 2 "KevinC@ppucc.io")
+	)
 	(junction
 		(at 64.77 121.285)
