File: Hardware/KiCAD/LED Board Rev 3/LEDboardRev3.kicad_sch (KiCad schematic)
At the start: 39 parts, among them J10 GND, J14 5V, J8 5V, J9 GND

Commit message: Added contact info and stuff to be super duper open source
Other:
- company: (none) -> Architeuthis Flux
- title: (none) -> LED Board Rev 3.1
